File: stusb.kicad_sch (KiCad schematic)
At the start: 24 parts, among them P1 USB_C_Plug, Q1 IRF8736, Q2 S8050, Q3 S8050, U4 STUSB4500QTR, U5 FT230XQ

Commit message: routed
Parts:
- added Q4: DTC143E, Package_TO_SOT_SMD:SOT-323_SC-70, symbol -Discrete:DTC143E
Connections:
- net at R7.1: now also Q4.3 (C); no longer U4.16 (VBUS_EN_SNK)
- new net: Q4.2 (E), U4.16 (VBUS_EN_SNK)
- new net power_en: Q4.1 (B)
Changed lines of the file:
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@@
     (stroke (width 0) (type solid) (color 0 0 0 0))
   )
-  (wire (pts (xy 181.61 76.2) (xy 196.85 76.2))
+  (wire (pts (xy 181.61 76.2) (xy 228.6 76.2))
     (stroke (width 0) (type solid) (color 0 0 0 0))
   )
@@
     (stroke (width 0) (type solid) (color 0 0 0 0))
   )
-  (wire (pts (xy 193.04 49.53) (xy 196.85 49.53))
+  (wire (pts (xy 193.04 49.53) (xy 228.6 49.53))
     (stroke (width 0) (type solid) (color 0 0 0 0))
   )
@@
     (stroke (width 0) (type solid) (color 0 0 0 0))
   )
-  (wire (pts (xy 196.85 76.2) (xy 196.85 49.53))
-    (stroke (width 0) (type solid) (color 0 0 0 0))
-  )
   (wire (pts (xy 209.55 20.32) (xy 209.55 25.4))
     (stroke (width 0) (type solid) (color 0 0 0 0))
@@
   )
   (wire (pts (xy 222.25 25.4) (xy 222.25 26.67))
+    (stroke (width 0) (type solid) (color 0 0 0 0))
+  )
+  (wire (pts (xy 228.6 49.53) (xy 228.6 57.15))
+    (stroke (width 0) (type solid) (color 0 0 0 0))
+  )
+  (wire (pts (xy 228.6 76.2) (xy 228.6 67.31))
     (stroke (width 0) (type solid) (color 0 0 0 0))
   )
@@
     (effects (font (size 1.27 1.27)) (justify left))
     (property "Intersheet References" "${INTERSHEET_REFS}" (id 0) (at 209.1328 151.0506 0)
+      (effects (font (size 1.27 1.27)) (justify left) hide)
+    )
+  )
+  (global_label "power_en" (shape input) (at 237.49 62.23 0)
+    (effects (font (size 1.27 1.27)) (justify left))
+    (property "Intersheet References" "${INTERSHEET_REFS}" (id 0) (at 250.1357 62.1506 0)
       (effects (font (size 1.27 1.27)) (justify left) hide)
     )
@@
     (pin "8")
   )
+  (symbol (lib_id "-Discrete:DTC143E") (at 231.14 62.23 0) (mirror y) (unit 1)
+    (in_bom yes) (on_board yes)
+    (property "Reference" "Q4" (id 0) (at 226.3648 61.0616 0)
+      (effects (font (size 1.27 1.27)) (justify left))
+    )
+    (property "Value" "DTC143E" (id 1) (at 226.3648 63.373 0)
+      (effects (font (size 1.27 1.27)) (justify left))
+    )
+    (property "Footprint" "Package_TO_SOT_SMD:SOT-323_SC-70" (id 2) (at 231.14 62.23 0)
+      (effects (font (size 1.27 1.27)) (justify left) hide)
+    )
+    (property "Datasheet" "" (id 3) (at 231.14 62.23 0)
+      (effects (font (size 1.27 1.27)) (justify left) hide)
+    )
+    (pin "1")
+    (pin "2")
+    (pin "3")
+  )
   (symbol (lib_id "Interface_USB:FT230XQ") (at 128.27 160.02 0) (unit 1)

Commit message: routing
Parts:
- renumbered C7 to C4, C8 to C6, C5 to C7, C9 to C8, C6 to C9, D11 to D10, D10 to D11, D9 to D12, D12 to D9, Q3 to Q1, Q4 to Q3, Q1 to Q4, R8 to R10, R4 to R2, R2 to R4, R9 to R5, R10 to R7, R7 to R8, R5 to R9, U5 to U3
Changed lines of the file:
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@@
   (symbol (lib_id "Device:D_Zener_Small") (at 116.84 31.75 270) (unit 1)
     (in_bom yes) (on_board yes)
-    (property "Reference" "D9" (id 0) (at 118.5672 30.5816 90)
+    (property "Reference" "D12" (id 0) (at 118.5672 30.5816 90)
       (effects (font (size 1.27 1.27)) (justify left))
     )
@@
   (symbol (lib_id "Device:D_Zener_Small") (at 222.25 29.21 270) (unit 1)
     (in_bom yes) (on_board yes)
-    (property "Reference" "D10" (id 0) (at 223.9772 28.0416 90)
+    (property "Reference" "D11" (id 0) (at 223.9772 28.0416 90)
       (effects (font (size 1.27 1.27)) (justify left))
     )
@@
   (symbol (lib_id "Device:R") (at 95.25 102.87 270) (unit 1)
     (in_bom yes) (on_board yes)
-    (property "Reference" "R2" (id 0) (at 96.52 105.41 0)
+    (property "Reference" "R4" (id 0) (at 96.52 105.41 0)
       (effects (font (size 1.27 1.27)) (justify left))
     )
@@
   (symbol (lib_id "Device:R") (at 156.21 35.56 180) (unit 1)
     (in_bom yes) (on_board yes)
-    (property "Reference" "R4" (id 0) (at 153.67 36.83 0)
+    (property "Reference" "R2" (id 0) (at 153.67 36.83 0)
       (effects (font (size 1.27 1.27)) (justify left))
     )
@@
   (symbol (lib_id "Device:R") (at 170.18 130.81 270) (unit 1)
     (in_bom yes) (on_board yes)
-    (property "Reference" "R9" (id 0) (at 171.45 133.35 0)
+    (property "Reference" "R5" (id 0) (at 171.45 133.35 0)
       (effects (font (size 1.27 1.27)) (justify left))
     )
@@
   (symbol (lib_id "Device:R") (at 170.18 146.05 270) (unit 1)
     (in_bom yes) (on_board yes)
-    (property "Reference" "R10" (id 0) (at 171.45 148.59 0)
+    (property "Reference" "R7" (id 0) (at 171.45 148.59 0)
       (effects (font (size 1.27 1.27)) (justify left))
     )
@@
   (symbol (lib_id "Device:R") (at 173.99 35.56 0) (unit 1)
     (in_bom yes) (on_board yes)
-    (property "Reference" "R5" (id 0) (at 176.53 34.29 0)
+    (property "Reference" "R9" (id 0) (at 176.53 34.29 0)
       (effects (font (size 1.27 1.27)) (justify left))
     )
@@
   (symbol (lib_id "Device:R") (at 189.23 49.53 270) (unit 1)
     (in_bom yes) (on_board yes)
-    (property "Reference" "R7" (id 0) (at 190.5 52.07 90)
+    (property "Reference" "R8" (id 0) (at 190.5 52.07 90)
       (effects (font (size 1.27 1.27)) (justify left))
     )
@@
   (symbol (lib_id "Device:R") (at 209.55 35.56 0) (unit 1)
     (in_bom yes) (on_board yes)
-    (property "Reference" "R8" (id 0) (at 212.09 34.29 0)
+    (property "Reference" "R10" (id 0) (at 212.09 34.29 0)
       (effects (font (size 1.27 1.27)) (justify left))
     )
@@
   (symbol (lib_id "Device:C") (at 106.68 172.72 0) (unit 1)
     (in_bom yes) (on_board yes)
-    (property "Reference" "C5" (id 0) (at 107.95 170.18 0)
+    (property "Reference" "C7" (id 0) (at 107.95 170.18 0)
       (effects (font (size 1.27 1.27)) (justify left))
     )
@@
   (symbol (lib_id "Device:C") (at 146.05 29.21 0) (unit 1)
     (in_bom yes) (on_board yes)
-    (property "Reference" "C6" (id 0) (at 149.86 27.94 0)
+    (property "Reference" "C9" (id 0) (at 149.86 27.94 0)
       (effects (font (size 1.27 1.27)) (justify left))
     )
@@
   (symbol (lib_id "Device:C") (at 185.42 59.69 270) (unit 1)
     (in_bom yes) (on_board yes)
-    (property "Reference" "C7" (id 0) (at 186.69 57.15 90)
+    (property "Reference" "C4" (id 0) (at 186.69 57.15 90)
       (effects (font (size 1.27 1.27)) (justify left))
     )
@@
   (symbol (lib_id "Device:C") (at 185.42 64.77 270) (unit 1)
     (in_bom yes) (on_board yes)
-    (property "Reference" "C8" (id 0) (at 186.69 68.58 90)
+    (property "Reference" "C6" (id 0) (at 186.69 68.58 90)
       (effects (font (size 1.27 1.27)) (justify left))
     )
@@
   (symbol (lib_id "Device:C") (at 196.85 35.56 0) (unit 1)
     (in_bom yes) (on_board yes)
-    (property "Reference" "C9" (id 0) (at 200.66 34.29 0)
+    (property "Reference" "C8" (id 0) (at 200.66 34.29 0)
       (effects (font (size 1.27 1.27)) (justify left))
     )
@@
   (symbol (lib_id "Power_Protection:SP0502BAHT") (at 73.66 118.11 0) (unit 1)
     (in_bom yes) (on_board yes)
-    (property "Reference" "D11" (id 0) (at 78.867 116.9416 0)
+    (property "Reference" "D10" (id 0) (at 78.867 116.9416 0)
       (effects (font (size 1.27 1.27)) (justify left))
     )
@@
   (symbol (lib_id "Power_Protection:SP0502BAHT") (at 113.03 86.36 0) (unit 1)
     (in_bom yes) (on_board yes)
-    (property "Reference" "D12" (id 0) (at 118.237 85.1916 0)
+    (property "Reference" "D9" (id 0) (at 118.237 85.1916 0)
       (effects (font (size 1.27 1.27)) (justify left))
     )
@@
   (symbol (lib_id "Transistor_BJT:S8050") (at 182.88 146.05 0) (unit 1)
     (in_bom yes) (on_board yes)
-    (property "Reference" "Q3" (id 0) (at 187.96 144.78 0)
+    (property "Reference" "Q1" (id 0) (at 187.96 144.78 0)
       (effects (font (size 1.27 1.27)) (justify left))
     )
@@
   (symbol (lib_id "Transistor_FET:FDS9435A") (at 181.61 27.94 270) (mirror x) (unit 1)
     (in_bom yes) (on_board yes)
-    (property "Reference" "Q1" (id 0) (at 181.61 19.2532 90))
+    (property "Reference" "Q4" (id 0) (at 181.61 19.2532 90))
     (property "Value" "IRF8736" (id 1) (at 181.61 21.5646 90))
     (property "Footprint" "Package_SO:SOIC-8_3.9x4.9mm_P1.27mm" (id 2) (at 179.705 22.86 0)
@@
   (symbol (lib_id "-Discrete:DTC143E") (at 231.14 62.23 0) (mirror y) (unit 1)
     (in_bom yes) (on_board yes)
-    (property "Reference" "Q4" (id 0) (at 226.3648 61.0616 0)
+    (property "Reference" "Q3" (id 0) (at 226.3648 61.0616 0)
       (effects (font (size 1.27 1.27)) (justify left))
     )
@@
   (symbol (lib_id "Interface_USB:FT230XQ") (at 128.27 160.02 0) (unit 1)
     (in_bom yes) (on_board yes)
-    (property "Reference" "U5" (id 0) (at 142.24 176.53 0))
+    (property "Reference" "U3" (id 0) (at 142.24 176.53 0))
     (property "Value" "FT230XQ" (id 1) (at 128.27 139.7 0)
       (effects (font (size 1.27 1.27)) hide)

Commit message: tweaks
Parts:
- Q4: footprint Package_SO:SOIC-8_3.9x4.9mm_P1.27mm -> precise:SOIC-8_3.9x4.9mm_P1.27mm
Changed lines of the file:
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@@
     (property "Reference" "Q4" (id 0) (at 181.61 19.2532 90))
     (property "Value" "IRF8736" (id 1) (at 181.61 21.5646 90))
-    (property "Footprint" "Package_SO:SOIC-8_3.9x4.9mm_P1.27mm" (id 2) (at 179.705 22.86 0)
+    (property "Footprint" "precise:SOIC-8_3.9x4.9mm_P1.27mm" (id 2) (at 179.705 22.86 0)
       (effects (font (size 1.27 1.27) italic) (justify left) hide)
     )

Commit message: sent to seeed
Parts:
- C7: value 100nf -> .1uf
- R3: footprint Capacitor_SMD:C_0603_1608Metric -> Resistor_SMD:R_0603_1608Metric
Changed lines of the file:
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@@
   (symbol (lib_id "Device:R") (at 95.25 102.87 270) (unit 1)
     (in_bom yes) (on_board yes)
-    (property "Reference" "R4" (id 0) (at 96.52 105.41 0)
+    (property "Reference" "R4" (id 0) (at 91.44 100.33 90)
       (effects (font (size 1.27 1.27)) (justify left))
     )
-    (property "Value" "27" (id 1) (at 93.98 105.41 0)
+    (property "Value" "27" (id 1) (at 95.25 100.33 90)
       (effects (font (size 1.27 1.27)) (justify left))
     )
@@
   (symbol (lib_id "Device:R") (at 95.25 107.95 270) (unit 1)
     (in_bom yes) (on_board yes)
-    (property "Reference" "R3" (id 0) (at 96.52 110.49 0)
+    (property "Reference" "R3" (id 0) (at 91.44 110.49 90)
       (effects (font (size 1.27 1.27)) (justify left))
     )
-    (property "Value" "27" (id 1) (at 93.98 110.49 0)
+    (property "Value" "27" (id 1) (at 95.25 110.49 90)
       (effects (font (size 1.27 1.27)) (justify left))
     )
-    (property "Footprint" "Capacitor_SMD:C_0603_1608Metric" (id 2) (at 95.25 106.172 90)
+    (property "Footprint" "Resistor_SMD:R_0603_1608Metric" (id 2) (at 95.25 106.172 90)
       (effects (font (size 1.27 1.27)) hide)
     )
@@
       (effects (font (size 1.27 1.27)) (justify left))
     )
-    (property "Value" "100nf" (id 1) (at 107.95 175.26 0)
+    (property "Value" ".1uf" (id 1) (at 107.95 175.26 0)
       (effects (font (size 1.27 1.27)) (justify left))
     )
