File: ws28xx.kicad_pcb (KiCad board)
At the start: 4 copper layers, 28.6 x 63.5 mm, 48 parts, among them J1 Conn_02x03_Odd_Even, J2 Conn_02x03_Odd_Even, P1 USB_C_Plug, Q1 IRF8736, Q2 S8050, Q3 S8050, SW1 en, SW2 io0, U0 ESP32-PICO-D4, U1 LM1117-3.3, U2 74AXP2T3407, U4 STUSB4500QTR, U5 FT230XQ

Commit message: routed
Parts:
- removed U2: 74AXP2T3407, precise:VSSOP-8_2.25x1.75mm_P0.5mm
- added Q4: DTC143E, Package_TO_SOT_SMD:SOT-323_SC-70, F.Cu at (127.5, 116.4)
- added R5: 100k, Resistor_SMD:R_0603_1608Metric, F.Cu at (130.2, 118.2)
- added U21: TXB0102, precise:SOIC-8, F.Cu at (123.2, 86.0)
- moved R4 1.42 mm to (131.5, 110.3)
- moved R6 0.35 mm to (133.2, 118.2)
Connections:
- U0 pad 18: unconnected-(U0-Pad18) -> power_en
- U4 pad 16: Net-(R7-Pad1) -> Net-(U4-Pad16)
Routing:
- net power_en: track 0.00 -> 25.3 mm, vias 0 -> 2
- net Net-(R8-Pad2): track 0.00 -> 22.6 mm, vias 0 -> 2
- net ESP_IO0: track 36.8 -> 52.5 mm
- net Net-(U4-Pad16): track 0.00 -> 7.87 mm
- net VDC: track 18.0 -> 25.8 mm, vias 1 -> 10
- net VBUS: track 17.9 -> 23.9 mm
- net Net-(Q1-Pad4): track 0.00 -> 5.03 mm
- net Net-(R7-Pad1): track 2.75 -> 6.58 mm
- net /LED_STRIP2: track 0.37 -> 3.60 mm
- net +3V3: track 5.60 -> 8.74 mm, vias 7 -> 8
- net /LED_STRIP1: track 0.40 -> 3.16 mm
- net Net-(JP3-Pad1): track 8.93 -> 11.2 mm
- net Net-(D12-Pad1): track 18.9 -> 20.8 mm, vias 1 -> 2
- net Net-(LEDS0-Pad2): track 18.7 -> 20.6 mm
- net /stat_led6: track 2.33 -> 0.77 mm
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- added copper zone on B.Cu, net VDC
- added copper zone on F.Cu, net VDC
Other:
- board size 28.6 x 63.5 mm -> 28.5 x 63.5 mm

Commit message: routed
Parts:
- renumbered C10 to C1, C11 to C3, C7 to C4, C12 to C5, C8 to C6, C5 to C7, C9 to C8, C6 to C9, D8 to D1, D11 to D10, D10 to D11, D9 to D12, D7 to D2, D5 to D3, D6 to D4, D4 to D5, D2 to D6, D1 to D7, D3 to D8, D12 to D9, J2 to J1, J1 to J2, JP3 to JP1, LEDS0 to LEDS1, LEDS1 to LEDS2, Q3 to Q1, Q4 to Q3, Q1 to Q4, R8 to R10, R4 to R2, R2 to R4, R9 to R5, R10 to R7, R7 to R8, R5 to R9, SW2 to SW1, SW1 to SW2, U21 to U1, U0 to U2, U5 to U3, U1 to U5
Routing:
- net VBUS: track 23.9 -> 26.8 mm
- net VDC: track 25.8 -> 27.1 mm, vias 10 -> 11
- net GND: track 28.1 -> 27.4 mm, vias 105 -> 110

Commit message: routing
Parts:
- added C10: 10uf, Capacitor_SMD:C_0805_2012Metric, B.Cu at (134.4, 94.2)
- C1: value C -> 470uf
- SW1, SW2: footprint Button_Switch_SMD:SW_Push_1P1T_NO_Vertical_Wuerth_434133025816 -> precise:SW_Push_1P1T_NO_Vertical
- moved LEDS1 53.2 mm to (170.0, 91.0), turned to 90 degrees
- moved LEDS2 50.3 mm to (170.0, 102.7), turned to 90 degrees
- moved JP1 42.4 mm to (161.8, 91.1), turned to 90 degrees
- moved SW2 39.8 mm to (113.4, 84.6), turned to 90 degrees
- moved AE1 36.7 mm to (149.0, 81.8), turned to 0 degrees
- moved J2 36.6 mm to (117.3, 83.8), turned to 0 degrees
- moved C1 35.9 mm to (159.6, 99.7), turned to 180 degrees
- moved C7 32.9 mm to (120.9, 84.4), turned to -90 degrees
- moved P1 31.2 mm to (114.8, 93.4), turned to -90 degrees
- moved C3 30.0 mm to (145.2, 85.0), turned to 180 degrees
- moved SW1 29.8 mm to (113.4, 102.1), turned to -90 degrees
- moved U3 29.1 mm to (124.4, 85.3), turned to 0 degrees
- moved U1 29.0 mm to (151.9, 90.3), turned to 180 degrees
- moved D4 27.9 mm to (153.0, 96.4), turned to 90 degrees
- moved Q1 27.8 mm to (129.1, 84.3), turned to 180 degrees
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Connections:
- D1 pad 1: GND -> Net-(D1-Pad1)
- D1 pad 2: Net-(D8-Pad2) -> +3V3
- D2 pad 1: GND -> Net-(D2-Pad1)
- D2 pad 2: Net-(D7-Pad2) -> +3V3
- D3 pad 1: GND -> Net-(D3-Pad1)
- D3 pad 2: Net-(D5-Pad2) -> +3V3
- D4 pad 1: GND -> Net-(D4-Pad1)
- D4 pad 2: Net-(D6-Pad2) -> +3V3
- D5 pad 1: GND -> Net-(D5-Pad1)
- D5 pad 2: Net-(D4-Pad2) -> +3V3
- D6 pad 1: GND -> Net-(D6-Pad1)
- D6 pad 2: Net-(D2-Pad2) -> +3V3
- D7 pad 1: GND -> Net-(D7-Pad1)
- D7 pad 2: Net-(D1-Pad2) -> +3V3
- D8 pad 1: GND -> Net-(D8-Pad1)
- D8 pad 2: Net-(D3-Pad2) -> +3V3
- RN1 pad 1: Net-(D1-Pad2) -> Net-(D7-Pad1)
- RN1 pad 10: unconnected-(RN1-Pad10) -> /stat_led6
- RN1 pad 2: Net-(D2-Pad2) -> Net-(D6-Pad1)
- RN1 pad 3: Net-(D3-Pad2) -> Net-(D8-Pad1)
- RN1 pad 4: Net-(D4-Pad2) -> Net-(D5-Pad1)
- RN1 pad 5: Net-(D5-Pad2) -> Net-(D3-Pad1)
- RN1 pad 6: Net-(D6-Pad2) -> Net-(D4-Pad1)
- RN1 pad 7: Net-(D7-Pad2) -> Net-(D2-Pad1)
- RN1 pad 8: Net-(D8-Pad2) -> Net-(D1-Pad1)
- U5 pad 3: VBUS -> VDC
Routing:
- net +3V3: track 8.74 -> 22.3 mm, vias 8 -> 11
- net VDC: track 27.1 -> 36.6 mm
- net Net-(D6-Pad2): track 6.71 -> 0.00 mm
- net Net-(D4-Pad1): track 0.00 -> 6.71 mm
- net Net-(D5-Pad2): track 6.09 -> 0.00 mm
- net Net-(D3-Pad1): track 0.00 -> 6.09 mm
- net Net-(D5-Pad1): track 0.00 -> 5.09 mm
- net Net-(D4-Pad2): track 5.09 -> 0.00 mm
- net Net-(D7-Pad2): track 4.46 -> 0.00 mm
- net Net-(D2-Pad1): track 0.00 -> 4.46 mm
- net Net-(D8-Pad1): track 0.00 -> 3.92 mm
- net Net-(D3-Pad2): track 3.92 -> 0.00 mm
- net Net-(D6-Pad1): track 0.00 -> 3.65 mm
- net Net-(D2-Pad2): track 3.65 -> 0.00 mm
- net Net-(D7-Pad1): track 0.00 -> 3.24 mm
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Other:
- board size 28.5 x 63.5 mm -> 63.5 x 28.5 mm
- board text added: "12v"
- board text added: "15v"
- board text added: "1a"
- board text added: "20v"
- board text added: "3+"
- board text added: "3a"
- board text added: "5v"
- board text added: "9v"

Commit message: -
Routing:
- net GND: track 28.0 -> 29.2 mm, vias 109 -> 111
Changed lines of the file:
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@@
     (pad "S1" thru_hole oval (at 4.32 -1.93) (locked) (size 2 0.9) (drill oval 1.7 0.6) (layers *.Cu *.Mask)
       (net 37 "GND") (pinfunction "SHIELD") (pintype "passive"))
-    (model "${KICAD6_3DMODEL_DIR}/Connector_USB.3dshapes/USB_C_Receptacle_Palconn_UTC16-G.wrl"
+    (model "${KICAD6_3DMODEL_DIR}/Connector_USB.3dshapes/USB_Micro-B_Molex_47346-0001.step"
       (offset (xyz 0 0 0))
       (scale (xyz 1 1 1))
@@
     (pad "2" smd rect (at 1.925 0.75 270) (size 1.25 0.9) (layers "F.Cu" "F.Paste" "F.Mask")
       (net 37 "GND") (pinfunction "2") (pintype "passive"))
-    (model "${KICAD6_3DMODEL_DIR}/Button_Switch_SMD.3dshapes/SW_Push_1P1T_NO_Vertical_Wuerth_434133025816.wrl"
+    (model "${KICAD6_3DMODEL_DIR}/Button_Switch_SMD.3dshapes/SW_SPST_TL3342.wrl"
       (offset (xyz 0 0 0))
       (scale (xyz 1 1 1))
@@
     (pad "2" smd rect (at 1.925 0.75 90) (size 1.25 0.9) (layers "F.Cu" "F.Paste" "F.Mask")
       (net 21 "ESP_EN") (pinfunction "2") (pintype "passive"))
-    (model "${KICAD6_3DMODEL_DIR}/Button_Switch_SMD.3dshapes/SW_Push_1P1T_NO_Vertical_Wuerth_434133025816.wrl"
+    (model "${KICAD6_3DMODEL_DIR}/Button_Switch_SMD.3dshapes/SW_SPST_TL3342.wrl"
       (offset (xyz 0 0 0))
       (scale (xyz 1 1 1))
@@
     (pad "8" smd rect (at -0.75 -1.55 180) (locked) (size 0.25 0.75) (layers "F.Cu" "F.Paste" "F.Mask")
       (net 22 "Net-(LEDS2-Pad2)") (pinfunction "B1") (pintype "bidirectional"))
+    (model "${KICAD6_3DMODEL_DIR}/Package_SO.3dshapes/SOIC-8_3.9x4.9mm_P1.27mm.wrl"
+      (offset (xyz 0 0 0))
+      (scale (xyz 1 1 1))
+      (rotate (xyz 0 0 90))
+    )
   )
   (footprint "Package_TO_SOT_SMD:SOT-23" (layer "F.Cu")
@@
   (segment (start 122.484997 85.663) (end 124.250387 85.663) (width 0.1778) (layer "F.Cu") (net 37))
   (segment (start 112.459997 83.913) (end 112.434997 83.938) (width 0.1778) (layer "F.Cu") (net 37))
+  (segment (start 133.737 101.313) (end 133.775 101.275) (width 0.1778) (layer "F.Cu") (net 37))
   (segment (start 133.959997 91.613002) (end 133.272908 92.300091) (width 0.1778) (layer "F.Cu") (net 37))
   (segment (start 112.659997 100.963) (end 112.734997 101.038) (width 0.1524) (layer "F.Cu") (net 37))
@@
   (segment (start 152.075 87.225) (end 152.075 88.725) (width 0.1778) (layer "F.Cu") (net 37))
   (segment (start 154.734997 94.138) (end 154.334997 94.07839) (width 0.1778) (layer "F.Cu") (net 37))
+  (segment (start 132.634997 101.313) (end 133.737 101.313) (width 0.1778) (layer "F.Cu") (net 37))
   (segment (start 116.509997 99.713) (end 115.834997 99.713) (width 0.1778) (layer "F.Cu") (net 37))
   (segment (start 127.059997 89.763) (end 127.284997 89.988) (width 0.1778) (layer "F.Cu") (net 37))
@@
   (via (at 112.434997 85.638) (size 0.6858) (drill 0.3302) (layers "F.Cu" "B.Cu") (net 37))
   (via (at 121.534997 84.488) (size 0.6858) (drill 0.3302) (layers "F.Cu" "B.Cu") (net 37))
+  (via (at 133.9 101.25) (size 0.6858) (drill 0.3302) (layers "F.Cu" "B.Cu") (net 37))
   (via (at 124.059997 92.563) (size 0.6858) (drill 0.3302) (layers "F.Cu" "B.Cu") (net 37))
   (via (at 137.859997 82.363) (size 0.6858) (drill 0.3302) (layers "F.Cu" "B.Cu") (net 37))
@@
   (via (at 124.434997 85.338) (size 0.6858) (drill 0.3302) (layers "F.Cu" "B.Cu") (net 37))
   (via (at 146.384997 91.288) (size 0.6858) (drill 0.3302) (layers "F.Cu" "B.Cu") (net 37))
+  (via (at 135.15 98.625) (size 0.6858) (drill 0.3302) (layers "F.Cu" "B.Cu") (net 37))
   (via (at 156.934997 82.988) (size 0.6858) (drill 0.3302) (layers "F.Cu" "B.Cu") (net 37))
   (via (at 152.584997 84.638) (size 0.6858) (drill 0.3302) (layers "F.Cu" "B.Cu") (net 37))
@@
     (polygon
       (pts
-        (xy 170.684997 81.938)
+        (xy 170.775 82.1)
         (xy 166.184997 85.738)
         (xy 159.484997 94.588)
         (xy 159.484997 101.763)
         (xy 138.584997 101.763)
+        (xy 133.3 101.85)
+        (xy 133.35 95.8)
+        (xy 138.463547 95.79718)
         (xy 138.307394 88.126668)
         (xy 149.332394 88.126668)
         (xy 149.858696 85.382334)
-        (xy 150.384997 82.638)
-        (xy 159.484997 82.688)
-      )
-    )
-  )
-  (zone (net 1) (net_name "VBUS") (layer "F.Cu") (hatch edge 0.508)
-    (connect_pads (clearance 0.508))
-    (min_thickness 0.254) (filled_areas_thickness no)
-    (fill yes (thermal_gap 0.508) (thermal_bridge_width 1.016))
-    (polygon
-      (pts
-        (xy 133.534997 103.238)
-        (xy 133.534997 93.138)
-        (xy 135.734997 93.138)
-        (xy 135.704276 103.24949)
+        (xy 150.6 82.1)
       )
     )
@@
         (xy 111.934997 82.188)
         (xy 146.184997 82.138)
-        (xy 146.184997 87.138)
+        (xy 146.2 87.2)
         (xy 153.834997 87.188)
         (xy 161.634997 84.638)
-        (xy 161.634997 82.688)
-        (xy 165.684997 81.888)
+        (xy 161.675 82.2)
         (xy 174.984997 82.188)
         (xy 174.984997 105.188)
@@
     (polygon
       (pts
-        (xy 153.684997 86.888)
-        (xy 146.534997 86.738)
-        (xy 146.534997 82.538)
-        (xy 161.184997 82.638)
-        (xy 161.184997 84.488)
-      )
-    )
-    (polygon
-      (pts
-        (xy 146.834997 87.188)
-        (xy 146.882916 87.178984)
-        (xy 146.884997 87.188)
+        (xy 161.35 82.175)
+        (xy 161.35 84.375)
+        (xy 153.825 86.75)
+        (xy 146.525 86.725)
+        (xy 146.525 82.15)
+        (xy 146.575 82.15)
       )
     )
@@
         (xy 111.384997 81.788)
         (xy 145.334997 81.738)
-        (xy 146.034997 82.688)
-        (xy 161.284997 82.838)
+        (xy 146.04016 82.16305)
+        (xy 161.29016 82.31305)
         (xy 165.534997 81.838)
         (xy 175.184997 81.788)

Commit message: tweaks
Parts:
- Q4: footprint Package_SO:SOIC-8_3.9x4.9mm_P1.27mm -> precise:SOIC-8_3.9x4.9mm_P1.27mm
Other:
- board text added: "precise.ai 2021 fastled_esp32_usb_pd"
Changed lines of the file:
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@@
-(kicad_pcb (version 20210126) (generator pcbnew)
+(kicad_pcb (version 20210228) (generator pcbnew)
   (general
     (thickness 4.69)
@@
       (dielectric_constraints no)
     )
+    (pad_to_mask_clearance 0)
     (aux_axis_origin 111.550997 105)
     (pcbplotparams
@@
     )
   )
-  (footprint "Package_SO:SOIC-8_3.9x4.9mm_P1.27mm" (layer "F.Cu")
+  (footprint "precise:SOIC-8_3.9x4.9mm_P1.27mm" (layer "F.Cu")
     (at 122.959992 101.412995 -90)
     (descr "SOIC, 8 Pin (JEDEC MS-012AA, https://www.analog.com/media/en/package-pcb-resources/package/pkg_pdf/soic_narrow-r/r_8.pdf), generated with kicad-footprint-generator ipc_gullwing_generator.py")
@@
     (property "Sheetname" "usb-pd")
     (attr smd)
-    (fp_text reference "Q4" (at 2.275 -3.375 90) (layer "F.SilkS")
+    (fp_text reference "Q4" (at 0 -3.4 -90) (layer "F.SilkS")
       (effects (font (size 1 1) (thickness 0.15)))
     )
-    (fp_text value "IRF8736" (at 0 3.4 90) (layer "F.Fab")
+    (fp_text value "IRF8736" (at 0 3.4 -90) (layer "F.Fab")
       (effects (font (size 1 1) (thickness 0.15)))
     )
-    (fp_text user "${REFERENCE}" (at 0 0 90) (layer "F.Fab")
+    (fp_text user "${REFERENCE}" (at 0 0 -90) (layer "F.Fab")
       (effects (font (size 0.98 0.98) (thickness 0.15)))
     )
@@
     (fp_line (start 0 -2.56) (end -3.45 -2.56) (layer "F.SilkS") (width 0.12))
     (fp_line (start 3.7 -2.7) (end -3.7 -2.7) (layer "F.CrtYd") (width 0.05))
-    (fp_line (start -3.7 2.7) (end 3.7 2.7) (layer "F.CrtYd") (width 0.05))
     (fp_line (start 3.7 2.7) (end 3.7 -2.7) (layer "F.CrtYd") (width 0.05))
     (fp_line (start -3.7 -2.7) (end -3.7 2.7) (layer "F.CrtYd") (width 0.05))
+    (fp_line (start -3.7 2.7) (end 3.7 2.7) (layer "F.CrtYd") (width 0.05))
+    (fp_line (start 1.95 -2.45) (end 1.95 2.45) (layer "F.Fab") (width 0.1))
     (fp_line (start 1.95 2.45) (end -1.95 2.45) (layer "F.Fab") (width 0.1))
+    (fp_line (start -0.975 -2.45) (end 1.95 -2.45) (layer "F.Fab") (width 0.1))
     (fp_line (start -1.95 -1.475) (end -0.975 -2.45) (layer "F.Fab") (width 0.1))
-    (fp_line (start 1.95 -2.45) (end 1.95 2.45) (layer "F.Fab") (width 0.1))
     (fp_line (start -1.95 2.45) (end -1.95 -1.475) (layer "F.Fab") (width 0.1))
-    (fp_line (start -0.975 -2.45) (end 1.95 -2.45) (layer "F.Fab") (width 0.1))
     (pad "1" smd roundrect (at -2.475 -1.905 270) (locked) (size 1.95 0.6) (layers "F.Cu" "F.Paste" "F.Mask") (roundrect_rratio 0.25)
-      (net 75 "VDC") (pinfunction "S") (pintype "passive"))
+      (net 75 "VDC") (pinfunction "S"))
     (pad "2" smd roundrect (at -2.475 -0.635 270) (locked) (size 1.95 0.6) (layers "F.Cu" "F.Paste" "F.Mask") (roundrect_rratio 0.25)
-      (net 75 "VDC") (pinfunction "S") (pintype "passive"))
+      (net 75 "VDC") (pinfunction "S"))
     (pad "3" smd roundrect (at -2.475 0.635 270) (locked) (size 1.95 0.6) (layers "F.Cu" "F.Paste" "F.Mask") (roundrect_rratio 0.25)
-      (net 75 "VDC") (pinfunction "S") (pintype "passive"))
+      (net 75 "VDC") (pinfunction "S"))
     (pad "4" smd roundrect (at -2.475 1.905 270) (locked) (size 1.95 0.6) (layers "F.Cu" "F.Paste" "F.Mask") (roundrect_rratio 0.25)
-      (net 26 "Net-(Q4-Pad4)") (pinfunction "G") (pintype "passive"))
+      (net 26 "Net-(Q4-Pad4)") (pinfunction "G"))
     (pad "5" smd roundrect (at 2.475 1.905 270) (locked) (size 1.95 0.6) (layers "F.Cu" "F.Paste" "F.Mask") (roundrect_rratio 0.25)
-      (net 1 "VBUS") (pinfunction "D") (pintype "passive"))
+      (net 1 "VBUS") (pinfunction "D"))
     (pad "6" smd roundrect (at 2.475 0.635 270) (locked) (size 1.95 0.6) (layers "F.Cu" "F.Paste" "F.Mask") (roundrect_rratio 0.25)
-      (net 1 "VBUS") (pinfunction "D") (pintype "passive"))
+      (net 1 "VBUS") (pinfunction "D"))
     (pad "7" smd roundrect (at 2.475 -0.635 270) (locked) (size 1.95 0.6) (layers "F.Cu" "F.Paste" "F.Mask") (roundrect_rratio 0.25)
-      (net 1 "VBUS") (pinfunction "D") (pintype "passive"))
+      (net 1 "VBUS") (pinfunction "D"))
     (pad "8" smd roundrect (at 2.475 -1.905 270) (locked) (size 1.95 0.6) (layers "F.Cu" "F.Paste" "F.Mask") (roundrect_rratio 0.25)
-      (net 1 "VBUS") (pinfunction "D") (pintype "passive"))
+      (net 1 "VBUS") (pinfunction "D"))
     (model "${KICAD6_3DMODEL_DIR}/Package_SO.3dshapes/SOIC-8_3.9x4.9mm_P1.27mm.wrl"
       (offset (xyz 0 0 0))
@@
     (fp_line (start -0.8 -0.4) (end 0.8 -0.4) (layer "F.Fab") (width 0.1))
     (pad "1" smd roundrect (at -0.775 0 270) (locked) (size 0.9 0.95) (layers "F.Cu" "F.Paste" "F.Mask") (roundrect_rratio 0.25)
-      (net 5 "Net-(C7-Pad1)"))
+      (net 5 "Net-(C7-Pad1)") (pintype "passive"))
     (pad "2" smd roundrect (at 0.775 0 270) (locked) (size 0.9 0.95) (layers "F.Cu" "F.Paste" "F.Mask") (roundrect_rratio 0.25)
-      (net 37 "GND"))
+      (net 37 "GND") (pintype "passive"))
     (model "${KICAD6_3DMODEL_DIR}/Capacitor_SMD.3dshapes/C_0603_1608Metric.wrl"
       (offset (xyz 0 0 0))
@@
   (gr_line (start 175.075 81.738003) (end 175.075 105) (layer "Edge.Cuts") (width 0.1))
   (gr_line (start 161.434997 76.488001) (end 145.684991 76.488001) (layer "Edge.Cuts") (width 0.09906))
+  (gr_text "precise.ai 2021 \nfastled_esp32_usb_pd" (at 143.125 87.375) (layer "B.SilkS")
+    (effects (font (size 2 2) (thickness 0.15)) (justify mirror))
+  )
   (gr_text "12v" (at 148.625 103.1 90) (layer "F.SilkS")
     (effects (font (size 1 1) (thickness 0.15)))
@@
   (segment (start 146.034997 97.656902) (end 146.034997 96.838) (width 0.1524) (layer "F.Cu") (net 87))
   (segment (start 125.272497 97.7255) (end 125.243277 97.69628) (width 0.1778) (layer "F.Cu") (net 88))
+  (segment (start 126.385983 98.938) (end 126.109997 98.925) (width 0.1778) (layer "F.Cu") (net 88))
   (segment (start 124.114124 97.69628) (end 122.334997 95.917153) (width 0.1778) (layer "F.Cu") (net 88))
-  (segment (start 126.109997 98.938) (end 126.109997 98.915225) (width 0.1778) (layer "F.Cu") (net 88))
-  (segment (start 126.385983 98.938) (end 126.109997 98.938) (width 0.1778) (layer "F.Cu") (net 88))
   (segment (start 127.172013 99.138802) (end 126.586785 99.138802) (width 0.1778) (layer "F.Cu") (net 88))
   (segment (start 125.243277 97.69628) (end 124.114124 97.69628) (width 0.1778) (layer "F.Cu") (net 88))
-  (segment (start 125.272497 97.7255) (end 125.209997 97.663) (width 0.1778) (layer "F.Cu") (net 88))
   (segment (start 125.525386 97.978389) (end 125.272497 97.7255) (width 0.1778) (layer "F.Cu") (net 88))
   (segment (start 127.48901 98.821805) (end 127.172013 99.138802) (width 0.1778) (layer "F.Cu") (net 88))

Commit message: sent to seeed
Routing:
- net GND: track 29.2 -> 30.1 mm
Other:
- board size 63.5 x 28.5 mm -> 63.5 x 29.5 mm
