File: ws28xx.kicad_sch (KiCad schematic)
At the start: 25 parts, among them J1 Conn_02x03_Odd_Even, J2 Conn_02x03_Odd_Even, SW1 en, SW2 io0, U0 ESP32-PICO-D4, U1 LM1117-3.3, U2 74AXP2T3407

Commit message: routed
Parts:
- removed U2: 74AXP2T3407, precise:VSSOP-8_2.25x1.75mm_P0.5mm, symbol precise:74AXP2T3407
- added U21: TXB0102, precise:SOIC-8, symbol precise:TXB0102
Connections:
- net +3V3: now also U21.3 (Vcca), U21.6 (OE)
- net GND: now also U21.2 (GND)
- net LED_STRIP1: now also U21.4 (A2)
- net LED_STRIP2: now also U21.5 (A1)
- net at JP3.1 (A): now also U21.7 (Vccb)
- net at LEDS1.2 (Pin_2): now also U21.8 (B1)
- net at LEDS0.2 (Pin_2): now also U21.1 (B2)
- net power_en: now reaches U0.18 (IO12)
Other:
- moved on the sheet: C10
Changed lines of the file:
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@@
   (junction (at 198.12 102.87) (diameter 0.9144) (color 0 0 0 0))
   (junction (at 203.2 102.87) (diameter 0.9144) (color 0 0 0 0))
-  (junction (at 238.76 142.24) (diameter 0.9144) (color 0 0 0 0))
+  (junction (at 217.17 132.08) (diameter 0.9144) (color 0 0 0 0))
   (junction (at 238.76 153.67) (diameter 0.9144) (color 0 0 0 0))
   (junction (at 242.57 134.62) (diameter 0.9144) (color 0 0 0 0))
@@
   (junction (at 245.11 129.54) (diameter 0.9144) (color 0 0 0 0))
   (junction (at 245.11 134.62) (diameter 0.9144) (color 0 0 0 0))
-  (junction (at 256.54 129.54) (diameter 0.9144) (color 0 0 0 0))
+  (junction (at 248.92 153.67) (diameter 0.9144) (color 0 0 0 0))
   (wire (pts (xy 24.13 153.67) (xy 24.13 158.75))
     (stroke (width 0) (type solid) (color 0 0 0 0))
@@
     (stroke (width 0) (type solid) (color 0 0 0 0))
   )
+  (wire (pts (xy 104.14 58.42) (xy 107.95 58.42))
+    (stroke (width 0) (type solid) (color 0 0 0 0))
+  )
   (wire (pts (xy 104.14 60.96) (xy 107.95 60.96))
     (stroke (width 0) (type solid) (color 0 0 0 0))
@@
     (stroke (width 0) (type solid) (color 0 0 0 0))
   )
-  (wire (pts (xy 217.17 129.54) (xy 217.17 134.62))
+  (wire (pts (xy 217.17 129.54) (xy 217.17 132.08))
+    (stroke (width 0) (type solid) (color 0 0 0 0))
+  )
+  (wire (pts (xy 217.17 132.08) (xy 217.17 134.62))
     (stroke (width 0) (type solid) (color 0 0 0 0))
   )
@@
     (stroke (width 0) (type solid) (color 0 0 0 0))
   )
-  (wire (pts (xy 238.76 142.24) (xy 238.76 153.67))
-    (stroke (width 0) (type solid) (color 0 0 0 0))
-  )
-  (wire (pts (xy 238.76 142.24) (xy 248.92 142.24))
-    (stroke (width 0) (type solid) (color 0 0 0 0))
-  )
   (wire (pts (xy 238.76 153.67) (xy 238.76 157.48))
     (stroke (width 0) (type solid) (color 0 0 0 0))
@@
     (stroke (width 0) (type solid) (color 0 0 0 0))
   )
-  (wire (pts (xy 240.03 135.89) (xy 240.03 137.16))
-    (stroke (width 0) (type solid) (color 0 0 0 0))
-  )
-  (wire (pts (xy 241.3 137.16) (xy 241.3 139.7))
-    (stroke (width 0) (type solid) (color 0 0 0 0))
-  )
-  (wire (pts (xy 241.3 139.7) (xy 238.76 139.7))
+  (wire (pts (xy 240.03 132.08) (xy 217.17 132.08))
+    (stroke (width 0) (type solid) (color 0 0 0 0))
+  )
+  (wire (pts (xy 240.03 137.16) (xy 240.03 132.08))
     (stroke (width 0) (type solid) (color 0 0 0 0))
   )
@@
     (stroke (width 0) (type solid) (color 0 0 0 0))
   )
-  (wire (pts (xy 242.57 134.62) (xy 242.57 146.05))
+  (wire (pts (xy 242.57 134.62) (xy 242.57 143.51))
     (stroke (width 0) (type solid) (color 0 0 0 0))
   )
@@
     (stroke (width 0) (type solid) (color 0 0 0 0))
   )
-  (wire (pts (xy 242.57 153.67) (xy 260.35 153.67))
+  (wire (pts (xy 242.57 151.13) (xy 242.57 153.67))
+    (stroke (width 0) (type solid) (color 0 0 0 0))
+  )
+  (wire (pts (xy 242.57 153.67) (xy 248.92 153.67))
     (stroke (width 0) (type solid) (color 0 0 0 0))
   )
@@
     (stroke (width 0) (type solid) (color 0 0 0 0))
   )
-  (wire (pts (xy 245.11 129.54) (xy 256.54 129.54))
+  (wire (pts (xy 245.11 129.54) (xy 260.35 129.54))
     (stroke (width 0) (type solid) (color 0 0 0 0))
   )
@@
     (stroke (width 0) (type solid) (color 0 0 0 0))
   )
-  (wire (pts (xy 246.38 135.89) (xy 240.03 135.89))
-    (stroke (width 0) (type solid) (color 0 0 0 0))
-  )
-  (wire (pts (xy 246.38 139.7) (xy 246.38 135.89))
-    (stroke (width 0) (type solid) (color 0 0 0 0))
-  )
-  (wire (pts (xy 246.38 146.05) (xy 256.54 146.05))
+  (wire (pts (xy 246.38 132.08) (xy 246.38 142.24))
+    (stroke (width 0) (type solid) (color 0 0 0 0))
+  )
+  (wire (pts (xy 246.38 132.08) (xy 260.35 132.08))
+    (stroke (width 0) (type solid) (color 0 0 0 0))
+  )
+  (wire (pts (xy 246.38 142.24) (xy 238.76 142.24))
     (stroke (width 0) (type solid) (color 0 0 0 0))
   )
@@
     (stroke (width 0) (type solid) (color 0 0 0 0))
   )
-  (wire (pts (xy 247.65 132.08) (xy 247.65 137.16))
-    (stroke (width 0) (type solid) (color 0 0 0 0))
-  )
-  (wire (pts (xy 247.65 137.16) (xy 241.3 137.16))
-    (stroke (width 0) (type solid) (color 0 0 0 0))
-  )
-  (wire (pts (xy 247.65 139.7) (xy 246.38 139.7))
+  (wire (pts (xy 247.65 139.7) (xy 238.76 139.7))
     (stroke (width 0) (type solid) (color 0 0 0 0))
   )
@@
     (stroke (width 0) (type solid) (color 0 0 0 0))
   )
-  (wire (pts (xy 248.92 134.62) (xy 248.92 142.24))
+  (wire (pts (xy 248.92 134.62) (xy 248.92 153.67))
     (stroke (width 0) (type solid) (color 0 0 0 0))
   )
@@
     (stroke (width 0) (type solid) (color 0 0 0 0))
   )
-  (wire (pts (xy 256.54 129.54) (xy 260.35 129.54))
-    (stroke (width 0) (type solid) (color 0 0 0 0))
-  )
-  (wire (pts (xy 256.54 146.05) (xy 256.54 129.54))
-    (stroke (width 0) (type solid) (color 0 0 0 0))
-  )
-  (wire (pts (xy 260.35 132.08) (xy 247.65 132.08))
+  (wire (pts (xy 248.92 153.67) (xy 260.35 153.67))
     (stroke (width 0) (type solid) (color 0 0 0 0))
   )
@@
     )
   )
+  (global_label "power_en" (shape input) (at 107.95 58.42 0)
+    (effects (font (size 1.27 1.27)) (justify left))
+    (property "Intersheet References" "${INTERSHEET_REFS}" (id 0) (at 120.5957 58.3406 0)
+      (effects (font (size 1.27 1.27)) (justify left) hide)
+    )
+  )
   (global_label "PWR_PDOK3" (shape input) (at 107.95 60.96 0)
     (effects (font (size 1.27 1.27)) (justify left))
@@
     (pin "2")
   )
-  (symbol (lib_id "Device:C") (at 242.57 149.86 0) (unit 1)
-    (in_bom yes) (on_board yes)
-    (property "Reference" "C10" (id 0) (at 246.38 148.59 0)
+  (symbol (lib_id "Device:C") (at 242.57 147.32 0) (unit 1)
+    (in_bom yes) (on_board yes)
+    (property "Reference" "C10" (id 0) (at 236.22 146.05 0)
       (effects (font (size 1.27 1.27)) (justify left))
     )
-    (property "Value" "C" (id 1) (at 246.38 151.13 0)
+    (property "Value" "C" (id 1) (at 246.38 148.59 0)
       (effects (font (size 1.27 1.27)) (justify left) hide)
     )
-    (property "Footprint" "Capacitor_SMD:C_Elec_10x10.2" (id 2) (at 243.535 153.67 0)
-      (effects (font (size 1.27 1.27)) hide)
-    )
-    (property "Datasheet" "~" (id 3) (at 242.57 149.86 0)
+    (property "Footprint" "Capacitor_SMD:C_Elec_10x10.2" (id 2) (at 243.535 151.13 0)
+      (effects (font (size 1.27 1.27)) hide)
+    )
+    (property "Datasheet" "~" (id 3) (at 242.57 147.32 0)
       (effects (font (size 1.27 1.27)) hide)
     )
@@
     (pin "3")
   )
-  (symbol (lib_id "precise:74AXP2T3407") (at 229.87 138.43 0) (unit 1)
-    (in_bom yes) (on_board yes)
-    (property "Reference" "U2" (id 0) (at 223.52 144.78 0))
-    (property "Value" "74AXP2T3407" (id 1) (at 227.33 130.81 0))
-    (property "Footprint" "precise:VSSOP-8_2.25x1.75mm_P0.5mm" (id 2) (at 228.6 152.4 0)
+  (symbol (lib_id "precise:TXB0102") (at 229.87 138.43 0) (unit 1)
+    (in_bom yes) (on_board yes)
+    (property "Reference" "U21" (id 0) (at 231.14 128.27 0))
+    (property "Value" "TXB0102" (id 1) (at 231.14 130.81 0))
+    (property "Footprint" "precise:SOIC-8" (id 2) (at 228.6 152.4 0)
       (effects (font (size 1.27 1.27)) hide)
     )
@@
       (reference "U1") (unit 1) (value "LM1117-3.3") (footprint "Package_TO_SOT_SMD:SOT-223")
     )
-    (path "/bec7aa6f-1fb1-44d5-8e09-bdc06ba71b7f"
-      (reference "U2") (unit 1) (value "74AXP2T3407") (footprint "precise:VSSOP-8_2.25x1.75mm_P0.5mm")
+    (path "/a3dd8c81-fcb0-4833-ba93-260fc4386d07"
+      (reference "U21") (unit 1) (value "TXB0102") (footprint "precise:SOIC-8")
     )
     (path "/47eee208-b208-4410-aeba-4ec25d1c9cd7/5f8b59f5-7c85-4c01-aea0-14825f3e1f25"
@@
       (reference "Q3") (unit 1) (value "S8050") (footprint "Package_TO_SOT_SMD:SOT-23")
     )
+    (path "/47eee208-b208-4410-aeba-4ec25d1c9cd7/b8d61184-dc23-43dd-a633-eae04bfa581c"
+      (reference "Q4") (unit 1) (value "DTC143E") (footprint "Package_TO_SOT_SMD:SOT-323_SC-70")
+    )
     (path "/47eee208-b208-4410-aeba-4ec25d1c9cd7/785e4899-e430-42d6-ab13-8025a2ef7099"

Commit message: routing
Parts:
- added C?: 10uf, Capacitor_SMD:C_0805_2012Metric, symbol Device:C
- C1: renamed from C10; value C -> 470uf
- SW1: renamed from SW2; footprint Button_Switch_SMD:SW_Push_1P1T_NO_Vertical_Wuerth_434133025816 -> precise:SW_Push_1P1T_NO_Vertical
- SW2: renamed from SW1; footprint Button_Switch_SMD:SW_Push_1P1T_NO_Vertical_Wuerth_434133025816 -> precise:SW_Push_1P1T_NO_Vertical
- renumbered C11 to C3, C12 to C5, D8 to D1, D7 to D2, D5 to D3, D6 to D4, D4 to D5, D2 to D6, D1 to D7, D3 to D8, J2 to J1, J1 to J2, JP3 to JP1, LEDS0 to LEDS1, LEDS1 to LEDS2, U21 to U1, U0 to U2, U1 to U5
Connections:
- net +3V3: now also D1.2 (A), D2.2 (A), D3.2 (A), D4.2 (A), D5.2 (A), D6.2 (A), D7.2 (A), D8.2 (A)
- net GND: now also C?.2; no longer D1.1 (K), D2.1 (K), D3.1 (K), D4.1 (K), D5.1 (K), D6.1 (K), D7.1 (K), D8.1 (K)
- net VBUS: no longer U5.3 (VI)
- net stat_led6: now also RN1.10 (R7.2)
- net at RN1.3 (R3.1): now also D8.1 (K); no longer D8.2 (A)
- net at RN1.1 (R1.1): now also D7.1 (K); no longer D7.2 (A)
- net at RN1.4 (R4.1): now also D5.1 (K); no longer D5.2 (A)
- net at RN1.7 (R7.1): now also D2.1 (K); no longer D2.2 (A)
- net at RN1.2 (R2.1): now also D6.1 (K); no longer D6.2 (A)
- net at RN1.6 (R6.1): now also D4.1 (K); no longer D4.2 (A)
- net at RN1.5 (R5.1): now also D3.1 (K); no longer D3.2 (A)
- net at RN1.8 (R8.1): now also D1.1 (K); no longer D1.2 (A)
- new net VDC: C?.1, U5.3 (VI)
Other:
- moved on the sheet: RN1

Commit message: -
Parts:
- gave numbers to parts that had none: 1
Changed lines of the file:
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@@
   (symbol (lib_id "Device:C") (at 30.48 168.91 0) (unit 1)
     (in_bom yes) (on_board yes)
-    (property "Reference" "C?" (id 0) (at 27.94 166.37 0)
+    (property "Reference" "C10" (id 0) (at 27.94 166.37 0)
       (effects (font (size 1.27 1.27)) (justify left))
     )
@@
     )
     (path "/7a5db98e-098b-4c8c-b059-352783143f13"
-      (reference "C?") (unit 1) (value "10uf") (footprint "Capacitor_SMD:C_0805_2012Metric")
+      (reference "C10") (unit 1) (value "10uf") (footprint "Capacitor_SMD:C_0805_2012Metric")
     )
     (path "/e699c72f-08fa-49a4-8e27-5620c6780b10"

Commit message: sent to seeed
Parts:
- C2: value C -> 1uf
- R1: value R -> 10k
- RN1: value R_Pack08 -> 330
Changed lines of the file:
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@@
     (effects (font (size 1.27 1.27)) (justify right bottom))
   )
-  (text "level translate\n" (at 234.95 149.86 180)
+  (text "level translate\n" (at 233.68 147.32 180)
     (effects (font (size 1.27 1.27)) (justify right bottom))
   )
@@
       (effects (font (size 1.27 1.27)) (justify left))
     )
-    (property "Value" "R" (id 1) (at 57.15 30.48 0)
+    (property "Value" "10k" (id 1) (at 57.15 30.48 0)
       (effects (font (size 1.27 1.27)) (justify left))
     )
@@
   (symbol (lib_id "Device:C") (at 34.29 41.91 90) (unit 1)
     (in_bom yes) (on_board yes)
-    (property "Reference" "C2" (id 0) (at 33.02 38.1 0)
-      (effects (font (size 1.27 1.27)) (justify left))
-    )
-    (property "Value" "C" (id 1) (at 35.56 38.1 0)
+    (property "Reference" "C2" (id 0) (at 34.29 45.72 90)
+      (effects (font (size 1.27 1.27)) (justify left))
+    )
+    (property "Value" "1uf" (id 1) (at 38.1 45.72 90)
       (effects (font (size 1.27 1.27)) (justify left))
     )
@@
       (effects (font (size 1.27 1.27)) (justify left))
     )
-    (property "Value" "470uf" (id 1) (at 246.38 148.59 0)
-      (effects (font (size 1.27 1.27)) (justify left) hide)
+    (property "Value" "470uf" (id 1) (at 236.22 149.86 0)
+      (effects (font (size 1.27 1.27)) (justify left))
     )
     (property "Footprint" "Capacitor_SMD:C_Elec_10x10.2" (id 2) (at 243.535 151.13 0)
@@
       (effects (font (size 1.27 1.27)) (justify left))
     )
-    (property "Value" "R_Pack08" (id 1) (at 187.96 95.25 0)
-      (effects (font (size 1.27 1.27)) (justify left) hide)
+    (property "Value" "330" (id 1) (at 187.96 95.25 0)
+      (effects (font (size 1.27 1.27)) (justify left))
     )
     (property "Footprint" "Resistor_SMD:R_Array_Convex_8x0602" (id 2) (at 186.055 96.52 90)
@@
     )
     (path "/d87f4c9d-1774-438d-90e9-a972eb7d0a40"
-      (reference "C2") (unit 1) (value "C") (footprint "Capacitor_SMD:C_0603_1608Metric")
+      (reference "C2") (unit 1) (value "1uf") (footprint "Capacitor_SMD:C_0603_1608Metric")
     )
     (path "/313890c0-83bd-4938-b24c-e14d95894b03"
@@
     )
     (path "/0312f4d6-fa3a-4cb9-8938-e1a91f425046"
-      (reference "R1") (unit 1) (value "R") (footprint "Resistor_SMD:R_0603_1608Metric")
+      (reference "R1") (unit 1) (value "10k") (footprint "Resistor_SMD:R_0603_1608Metric")
     )
     (path "/d24bd43c-0cd7-465f-8e38-700d1e6dac2b"
-      (reference "RN1") (unit 1) (value "R_Pack08") (footprint "Resistor_SMD:R_Array_Convex_8x0602")
+      (reference "RN1") (unit 1) (value "330") (footprint "Resistor_SMD:R_Array_Convex_8x0602")
     )
     (path "/36fdb679-e63b-4b2d-b8f9-b8363bc1aa92"
@@
     )
     (path "/47eee208-b208-4410-aeba-4ec25d1c9cd7/8ac962f1-1642-4e9f-83d3-3c58e79c15f9"
-      (reference "C7") (unit 1) (value "100nf") (footprint "Capacitor_SMD:C_0603_1608Metric")
+      (reference "C7") (unit 1) (value ".1uf") (footprint "Capacitor_SMD:C_0603_1608Metric")
     )
     (path "/47eee208-b208-4410-aeba-4ec25d1c9cd7/82fdb6fd-ccbc-419a-bdcd-08ee1a69dd59"
@@
     )
     (path "/47eee208-b208-4410-aeba-4ec25d1c9cd7/291b2f36-195f-471d-8b62-16d228259ace"
-      (reference "R3") (unit 1) (value "27") (footprint "Capacitor_SMD:C_0603_1608Metric")
+      (reference "R3") (unit 1) (value "27") (footprint "Resistor_SMD:R_0603_1608Metric")
     )
     (path "/47eee208-b208-4410-aeba-4ec25d1c9cd7/785e4899-e430-42d6-ab13-8025a2ef7099"
